File: Hardware/Yet-Another-Nixie-Clock/Yet-Another-Nixie-Clock.kicad_sch (KiCad schematic)
At the start: 8 parts, among them Q1 BF820, Q2 Q_NMOS, U1 ESP32-C3-WROOM-02, U2 74HC595, U3 MAX1771xSA

Commit message: Schematic advancements
Parts:
- removed C1: 4.7uF / 250V, Capacitor_SMD:C_Elec_8x10.2, symbol Device:C_Small_US
- removed L1: 100uH / 2.5 A, Inductor_SMD:L_APV_APH0840, symbol Device:L_Small
- removed Q1: BF820, Package_TO_SOT_SMD:TSOT-23, symbol Transistor_BJT:Q_NPN_BCE
- removed Q2: Q_NMOS, Package_TO_SOT_SMD:TO-263-2, symbol Transistor_FET:Q_NMOS_DGS
- removed R1: R_Small_US, symbol Device:R_Small_US
- removed U1: ESP32-C3-WROOM-02, RF_Module:ESP32-C3-WROOM-02, symbol RF_Module:ESP32-C3-WROOM-02
- removed U2: 74HC595, Package_SO:SOIC-16_3.9x9.9mm_P1.27mm, symbol 74xx:74HC595
- removed U3: MAX1771xSA, Package_SO:SO-8_3.9x4.9mm_P1.27mm, symbol Regulator_Switching:MAX1771xSA
- added C10, C11, C7: 22uF, Capacitor_SMD:C_0603_1608Metric, symbol Device:C_Small
- added C6: 100nF, Capacitor_SMD:C_0603_1608Metric, symbol Device:C_Small
- added C8, C9: 10uF, Capacitor_SMD:C_0603_1608Metric, symbol Device:C_Small
- added D2: Green, LED_SMD:LED_0603_1608Metric, symbol Device:LED
- added J1: PJ-002BH, Yet-Another-Nixie-Clock:CUI_PJ-002BH, symbol Connector:Barrel_Jack_Switch
- added L2: 22uH, Inductor_SMD:L_APV_APH0615, symbol Device:L_Small
- added R5: 33.2k, symbol Device:R_Small_US
- added R6: 10k, symbol Device:R_Small_US
- added R7: 1k, symbol Device:R_Small_US
- added U4: TPS563200, Package_TO_SOT_SMD:SOT-23-6, symbol Regulator_Switching:TPS563200
- added U5: ESP32-WROOM-32, RF_Module:ESP32-WROOM-32, symbol RF_Module:ESP32-WROOM-32
Connections:
- net GND: now also C10.2, C11.2, C7.2, C8.2, C9.2, D2.1 (K), J1.2, R6.2, U4.1 (GND), U5.1 (GND), U5.15 (GND), U5.38 (GND), U5.39 (GND)
- new net: C6.1, U4.6 (VBST)
- new net: C6.2, L2.1, U4.2 (SW)
- new net: D2.2 (A), R7.1
- new net: R5.2, R6.1, U4.4 (VFB)
- new net VCC12V: C8.1, C9.1, J1.1, U4.3 (VIN), U4.5 (EN)
- new net VCC3V3: C10.1, C11.1, C7.1, L2.2, R5.1, R7.2, U5.2 (VDD)
Other:
- added sheet HV PSU (sch/hv_psu.kicad_sch)
- added sheet Nixie Driver (sch/nixie_driver.kicad_sch)
- note added: "https://www.electronics-lab.com/project/hv-nixie-dc-dc-switching-power-supply/ https://github.com/marcinsaj/IN12-IN15-Binary-Nixie-Clock/blob/master/datasheet/Nixie-Tube-Driver-V2-Schematic.pdf https://gra-afch.com/how-it-works/how-to-drive-a-nixie-tubes/"
- note removed: "https://www.electronics-lab.com/project/hv-nixie-dc-dc-switching-power-supply/ https://github.com/marcinsaj/IN12-IN15-Binary-Nixie-Clock/blob/master/datasheet/Nixie-Tube-Driver-V2-Schematic.pdf"

Commit message: Schematic work
Parts:
- added BT1: Battery_Cell, symbol Device:Battery_Cell
- added C12, C16: 10uF, Capacitor_SMD:C_0603_1608Metric, symbol Device:C_Small
- added C13, C14, C15, C17, C18, C19: 100nF, Capacitor_SMD:C_0603_1608Metric, symbol Device:C_Small
- added J3: JTAG, symbol Connector_Generic:Conn_02x05_Odd_Even
- added J6: USB_C_Receptacle_USB2.0, Connector_USB:USB_C_Receptacle_HCTL_HC-TYPE-C-16P-01A, symbol Connector:USB_C_Receptacle_USB2.0
- added Q1, Q3: MMBT2222A, Package_TO_SOT_SMD:SOT-23, symbol Transistor_BJT:MMBT2222A
- added R1, R8, R9: 10k, symbol Device:R_Small_US
- added R11: 100k, Resistor_SMD:R_0402_1005Metric, symbol Device:R_Small_US
- added R12: 330, Resistor_SMD:R_0402_1005Metric, symbol Device:R_Small_US
- added R13, R14: 5.1k, Resistor_SMD:R_0402_1005Metric, symbol Device:R_Small_US
- added R15, R16: 4.7k, Resistor_SMD:R_0402_1005Metric, symbol Device:R_Small_US
- added R20: 0, Resistor_SMD:R_0402_1005Metric, symbol Device:R_Small_US
- added U12: USBLC6-2P6, Package_TO_SOT_SMD:SOT-666, symbol Power_Protection:USBLC6-2P6
- added U13: DS3231M, Package_SO:SOIC-16W_7.5x10.3mm_P1.27mm, symbol Timer_RTC:DS3231M
- added U14: CP2102N-Axx-xQFN24, Package_DFN_QFN:QFN-24-1EP_4x4mm_P0.5mm_EP2.6x2.6mm, symbol Interface_USB:CP2102N-Axx-xQFN24
Connections:
- net GND: now also BT1.2 (-), C12.2, C13.1, C14.1, C15.1, C16.2, C17.1, C18.1, C19.1, J3.3 (Pin_3), J3.5 (Pin_5), J3.7 (Pin_7), J3.9 (Pin_9), J6.A1 (GND), J6.A12 (GND), J6.B1 (GND), J6.B12 (GND), J6.S1 (SHIELD), R13.2, R14.2, U12.2 (GND), U13.10 (GND), U13.11 (GND), U13.12 (GND), U13.13 (GND), U13.5 (GND), U13.6 (GND), U13.7 (GND), U13.8 (GND), U13.9 (GND), U14.2 (GND), U14.25 (GND)
- net VCC3V3: now also C19.2, R11.1, R15.1, R16.1, R20.1, U13.2 (VCC)
- net ESP_TMS: now reaches U5.13 (IO14)
- net ESP_TMS: now also J3.2 (Pin_2)
- net ESP_TDI: now reaches U5.14 (IO12)
- net ESP_TDI: now also J3.8 (Pin_8)
- net ESP_TCK: now reaches U5.16 (IO13)
- net ESP_TCK: now also J3.4 (Pin_4)
- net ESP_TDO: now reaches U5.23 (IO15)
- net ESP_TDO: now also J3.6 (Pin_6)
- net IO0: now reaches U5.25 (IO0)
- net IO0: now also Q1.3 (C)
- net ESP_RST: now reaches U5.3 (EN)
- net ESP_RST: now also Q3.3 (C), R12.2
- net RTC_SDA: now reaches U5.33 (IO21)
- net RTC_SDA: now also R16.2, U13.15 (SDA)
- net CP_TXD: now reaches U5.34 (RXD0/IO3)
- net CP_TXD: now also U14.21 (TXD)
- net CP_RXD: now reaches U5.35 (TXD0/IO1)
- net CP_RXD: now also U14.20 (RXD)
- net RTC_SCL: now reaches U5.36 (IO22)
- net RTC_SCL: now also R15.2, U13.16 (SCL)
- new net: J6.B5 (CC2), R13.1
- new net: R9.2, U14.9 (~{RST})
- new net: C17.2, R11.2, R12.1
- new net: Q3.1 (B), R8.2
- new net: J6.A5 (CC1), R14.1
- new net: J3.1 (Pin_1), R20.2
- new net: Q1.1 (B), R1.2
- new net CP_3V3: C12.1, C13.2, R9.1, U14.5 (VIO), U14.6 (VDD)
- new net CP_~{CTS}: U14.18 (~{CTS})
- new net CP_~{DSR}: U14.22 (~{DSR})
- new net CP_~{DTR}: Q1.2 (E), R8.1, U14.23 (~{DTR})
- new net CP_~{RTS}: Q3.2 (E), R1.1, U14.19 (~{RTS})
- new net RTC_SQW: U13.3 (~{INT}/SQW)
- new net USB_D_N: U12.6 (I/O1), U14.4 (D-)
- new net USB_D_P: U12.4 (I/O2), U14.3 (D+)
- new net USB_D_RAW_N: J6.A7 (D-), J6.B7 (D-), U12.1 (I/O1)
- new net USB_D_RAW_P: J6.A6 (D+), J6.B6 (D+), U12.3 (I/O2)
- new net VBAT: BT1.1 (+), C18.2, U13.14 (VBAT)
- new net VBUS: C14.2, C15.2, C16.1, J6.A4 (VBUS), J6.A9 (VBUS), J6.B4 (VBUS), J6.B9 (VBUS), U12.5 (VBUS), U14.7 (VREGIN), U14.8 (VBUS)
- no-connect marks 0 -> 3
Other:
- moved on the sheet: U5

Commit message: Schematic work
Other:
- removed sheet HV PSU
- sheet Nixie Driver ports: added G_A[0..5], N[0..3], ~{N_LE}; removed none
- moved on the sheet: BT1, C10, C11, C12, C13, C14, C15, C16, C17, C18, C19, C6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

Commit message: Schematic work and fixes
Parts:
- added D2: LED_RGB, OpenTama:LED_RGB_TC5050, symbol Device:LED_RGB
- added R10, R9: 1k, symbol Device:R_Small_US
- added R13, R17: 10k, symbol Device:R_Small_US
- added SW1, SW2, SW3: SW_MEC_5E, Yet-Another-Nixie-Clock:SW_SKRPACE010, symbol Switch:SW_MEC_5E
- R11: value 100k -> 1k; footprint Resistor_SMD:R_0402_1005Metric -> (none); LCSC C25803 -> C22548
- R12: value 330 -> 10k; footprint Resistor_SMD:R_0402_1005Metric -> (none); LCSC C105875 -> C98220
- renumbered C9 to C1, C17 to C12, C19 to C13, C18 to C14, C8 to C2, C6 to C3, C15 to C4, C14 to C5, C16 to C6, C13 to C7, C12 to C8, C7 to C9, D2 to D1, J6 to J2, L2 to L1, Q3 to Q2, R15 to R14, R16 to R15, R20 to R16, R8 to R2, R9 to R3, R13 to R4, R14 to R5, R5 to R6, R6 to R7, R7 to R8, U14 to U1, U4 to U2, U12 to U3, U13 to U4
Connections:
- net ESP_RST: now also C12.2, SW1.3 (K), SW1.4 (A)
- net GND: now also D2.1 (RK), D2.2 (GK), D2.3 (BK), SW1.1, SW1.2, SW2.1, SW2.2, SW3.1, SW3.2
- net IO0: now also R13.2, SW2.3 (K), SW2.4 (A)
- net VCC3V3: now also R12.1, R13.1, R17.1; no longer R11.1
- net G_A0: now reaches U5.10 (IO25)
- net G_A1: now reaches U5.11 (IO26)
- net G_A2: now reaches U5.12 (IO27)
- net LED_R: now reaches U5.24 (IO2)
- net LED_R: now also R9.1
- net LED_G: now reaches U5.26 (IO4)
- net LED_G: now also R10.1
- net N0: now reaches U5.27 (IO16)
- net N1: now reaches U5.28 (IO17)
- net LED_B: now reaches U5.29 (IO5)
- net LED_B: now also R11.1
- net N2: now reaches U5.30 (IO18)
- net N3: now reaches U5.31 (IO19)
- net SW1: now reaches U5.37 (IO23)
- net SW1: now also R17.2, SW3.3 (K), SW3.4 (A)
- net G_A5: now reaches U5.6 (IO34)
- net ~{N_LE}: now reaches U5.7 (IO35)
- net G_A3: now reaches U5.8 (IO32)
- net G_A4: now reaches U5.9 (IO33)
- new net: D2.5 (GA), R10.2
- new net: D2.4 (BA), R11.2
- new net: D2.6 (RA), R9.2
Other:
- moved on the sheet: C1, C10, C11, C2, C3, C9, D1, J1, L1, R6, R7, R8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
