File: Hardware/Yet-Another-Nixie-Clock/Yet-Another-Nixie-Clock.kicad_pcb (KiCad board)
At the start: 2 copper layers, 87 parts, among them J1 PJ-002BH, J2 USB_C_Receptacle_USB2.0, J4 Nixie IN12, J5 Nixie IN12, J6 Nixie IN12, J7 Nixie IN12, J8 Nixie IN12, J9 Nixie IN12, Q1 MMBT2222A, Q10 BF820, Q11 BF820, Q12 BF820, Q13 BF820, Q14 BF820, Q15 BF820, Q16 PMBTA42, Q17 PMBTA92, Q18 PMBTA42, Q19 PMBTA92, Q2 MMBT2222A, Q20 PMBTA42, Q21 PMBTA92, Q22 PMBTA42, Q23 PMBTA92, Q24 PMBTA42, Q25 PMBTA92, Q3 Q_NMOS, Q4 PMBTA42, Q5 PMBTA92, Q6 BF820, Q7 BF820, Q8 BF820, Q9 BF820, SW1 SW_MEC_5E, SW2 SW_MEC_5E, SW3 SW_MEC_5E, U1 CP2102N-Axx-xQFN24, U2 TPS563200, U3 USBLC6-2P6, U4 DS3231M, U5 ESP32-WROOM-32, U6 MAX1771xSA

Commit message: Schematic advancements, separated boards
Parts:
- added D15: LED, LED_SMD:LED_0603_1608Metric, F.Cu at (216.9, 39.0)
- added D16: LED, LED_SMD:LED_0603_1608Metric, F.Cu at (216.9, 41.6)
- added D17: LED, LED_SMD:LED_0603_1608Metric, F.Cu at (216.9, 44.2)
- added D2: LED, LED_SMD:LED_0603_1608Metric, F.Cu at (216.9, 36.4)
- added H1: MountingHole_Pad, MountingHole:MountingHole_3.2mm_M3_Pad, F.Cu at (59.6, 73.2)
- added H2: MountingHole_Pad, MountingHole:MountingHole_3.2mm_M3_Pad, F.Cu at (243.6, 73.2)
- added H3: MountingHole_Pad, MountingHole:MountingHole_3.2mm_M3_Pad, F.Cu at (243.6, 127.2)
- added H4: MountingHole_Pad, MountingHole:MountingHole_3.2mm_M3_Pad, F.Cu at (59.6, 127.2)
- added J10: Conn_02x06_Odd_Even, Connector_PinHeader_2.54mm:PinHeader_2x06_P2.54mm_Vertical_SMD, B.Cu at (243.6, 113.2)
- added J11: Conn_02x06_Odd_Even, Connector_PinHeader_2.54mm:PinHeader_2x06_P2.54mm_Vertical_SMD, B.Cu at (229.6, 127.2)
- added R21: 4.7k, Resistor_SMD:R_0603_1608Metric, B.Cu at (233.8, 98.7)
- added R22: 300k, Resistor_SMD:R_0603_1608Metric, B.Cu at (240.1, 99.4)
- added R23: 10k, Resistor_SMD:R_0603_1608Metric, B.Cu at (240.1, 102.5)
- added R24: 4.7k, Resistor_SMD:R_0603_1608Metric, B.Cu at (233.8, 102.3)
- added R25: 10k, Resistor_SMD:R_0603_1608Metric, B.Cu at (247.5, 86.2)
- added R26: 10k, Resistor_SMD:R_0603_1608Metric, B.Cu at (245.9, 86.2)
- added R27: 4.7k, Resistor_SMD:R_0603_1608Metric, B.Cu at (209.5, 106.0)
- added R28: 300k, Resistor_SMD:R_0603_1608Metric, B.Cu at (209.9, 100.1)
- added R29: 10k, Resistor_SMD:R_0603_1608Metric, B.Cu at (213.0, 100.1)
- added R30: 4.7k, Resistor_SMD:R_0603_1608Metric, B.Cu at (212.9, 106.0)
- added R31: 4.7k, Resistor_SMD:R_0603_1608Metric, B.Cu at (179.8, 106.2)
- added R32: 300k, Resistor_SMD:R_0603_1608Metric, B.Cu at (180.1, 100.2)
- added R33: 10k, Resistor_SMD:R_0603_1608Metric, B.Cu at (183.2, 100.2)
- added R34: 4.7k, Resistor_SMD:R_0603_1608Metric, B.Cu at (182.9, 106.2)
- added R35: 4.7k, Resistor_SMD:R_0603_1608Metric, B.Cu at (150.0, 105.7)
- added R36: 300k, Resistor_SMD:R_0603_1608Metric, B.Cu at (150.1, 99.7)
- added R37: 10k, Resistor_SMD:R_0603_1608Metric, B.Cu at (153.2, 99.7)
- added R38: 4.7k, Resistor_SMD:R_0603_1608Metric, B.Cu at (153.1, 105.7)
- added R39: 4.7k, Resistor_SMD:R_0603_1608Metric, B.Cu at (119.9, 105.5)
- added R40: 300k, Resistor_SMD:R_0603_1608Metric, B.Cu at (120.0, 99.5)
- added R41: 10k, Resistor_SMD:R_0603_1608Metric, B.Cu at (123.0, 99.5)
- added R42: 4.7k, Resistor_SMD:R_0603_1608Metric, B.Cu at (123.0, 105.5)
- added R43: 4.7k, Resistor_SMD:R_0603_1608Metric, B.Cu at (90.0, 106.0)
- added R44: 300k, Resistor_SMD:R_0603_1608Metric, B.Cu at (90.2, 100.3)
- added R45: 10k, Resistor_SMD:R_0603_1608Metric, B.Cu at (93.3, 100.3)
- added R46: 4.7k, Resistor_SMD:R_0603_1608Metric, B.Cu at (93.0, 106.0)
- added RN1: R_Pack08_Split, Yet-Another-Nixie-Clock:RES-ARRAY-SMD_0402-16P-L4.0-W1.6-BL-2, B.Cu at (239.4, 85.8)
- added U7: 74HC237, Package_SO:TSSOP-16_4.4x5mm_P0.65mm, B.Cu at (240.5, 92.3)
- added U8: 74HC237, Package_SO:TSSOP-16_4.4x5mm_P0.65mm, B.Cu at (246.2, 92.3)
- Q10, Q11, Q12, Q13, Q14, Q15, Q16, Q18, Q20, Q22, Q24, Q4, Q6, Q7, Q8, Q9, U5: moved to B.Cu
- Q17, Q19, Q21, Q23, Q25, Q5: footprint Package_TO_SOT_SMD:TSOT-23 -> Package_TO_SOT_SMD:SOT-23; moved to B.Cu
- moved C15 323.8 mm to (-44.6, 146.7)
- moved D3 323.8 mm to (-44.5, 152.4)
- moved Q3 323.8 mm to (-56.7, 129.3)
- moved U2 323.8 mm to (-96.1, 62.0)
- moved C1 323.8 mm to (-145.7, 65.6)
- moved C10 323.8 mm to (-141.7, 75.7)
- moved C11 323.8 mm to (-137.7, 65.6)
- moved C12 323.8 mm to (-137.7, 68.2)
- moved C13 323.8 mm to (-137.7, 70.7)
- moved C14 323.8 mm to (-137.7, 73.2)
- moved C16 323.8 mm to (-52.2, 150.9)
- moved C17 323.8 mm to (-52.2, 153.4)
- moved C18 323.8 mm to (-60.8, 140.4)
- moved C19 323.8 mm to (-46.9, 125.2)
- moved C2 323.8 mm to (-145.7, 68.2)
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Connections:
- net /LED_B renamed /LED_2
- net /LED_G renamed /LED_1
- net /LED_R renamed /LED_3
Routing:
- net /Nixie Driver/K9: track 0.00 -> 348.8 mm, vias 0 -> 6
- net /Nixie Driver/K8: track 0.00 -> 296.4 mm, vias 0 -> 6
- net /Nixie Driver/K3: track 0.00 -> 272.1 mm, vias 0 -> 6
- net /Nixie Driver/K7: track 0.00 -> 259.3 mm, vias 0 -> 6
- net /Nixie Driver/K4: track 0.00 -> 247.5 mm, vias 0 -> 6
- net /Nixie Driver/K6: track 0.00 -> 240.3 mm, vias 0 -> 6
- net /Nixie Driver/K5: track 0.00 -> 234.0 mm, vias 0 -> 6
- net /Nixie Driver/K0: track 0.00 -> 226.8 mm, vias 0 -> 6
- net /Nixie Driver/K2: track 0.00 -> 221.5 mm, vias 0 -> 6
- net /Nixie Driver/K1: track 0.00 -> 202.7 mm, vias 0 -> 6
- net /G_A5: track 0.00 -> 188.8 mm, vias 0 -> 2
- net /G_A4: track 0.00 -> 145.9 mm, vias 0 -> 2
- net /G_A3: track 0.00 -> 117.5 mm, vias 0 -> 2
- net /G_A2: track 0.00 -> 89.5 mm, vias 0 -> 2
- net /G_A1: track 0.00 -> 61.4 mm, vias 0 -> 2
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Other:
- board outline added: 200 x 70 mm
- copper layers 2 -> 4
