File: Hardware/Yet-Another-Nixie-Clock/sch/hv_psu.kicad_sch (KiCad schematic)
At the start: 13 parts, among them Q2 Q_NMOS, U3 MAX1771xSA

Commit message: Schematic work
Parts:
- renumbered C3 to C1, C4 to C2, C2 to C3, C1 to C4, U3 to U1

Commit message: Schematic work and fixes
Other:
- moved on the sheet: C1, C2, C3, C4, C5, D1, L1, Q2, R2, R3, R4, RV1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

Commit message: Schematic work and fixes
Parts:
- renumbered C1 to C15, C2 to C16, C3 to C17, C4 to C18, C5 to C19, D1 to D3, L1 to L2, Q2 to Q3, R2 to R18, R3 to R19, R4 to R20, U1 to U6
Changed lines of the file:
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@@
 		(dnp no)
 		(fields_autoplaced yes)
-		(property "Reference" "R2"
+		(property "Reference" "R18"
 			(at 163.83 99.0599 0)
 			(effects
@@
 			(project "Yet-Another-Nixie-Clock"
 				(path "/78ce616d-4594-460a-a6b5-d8dd90d9a741/3fd9b30e-c53f-44d4-9eb4-8fd367607a00/50401da1-09e6-4577-9a0a-561e17376ad4"
-					(reference "R2")
+					(reference "R18")
 					(unit 1)
 				)
@@
 		(dnp no)
 		(fields_autoplaced yes)
-		(property "Reference" "#PWR09"
+		(property "Reference" "#PWR059"
 			(at 184.15 119.38 0)
 			(effects
@@
 			(project "Yet-Another-Nixie-Clock"
 				(path "/78ce616d-4594-460a-a6b5-d8dd90d9a741/3fd9b30e-c53f-44d4-9eb4-8fd367607a00/50401da1-09e6-4577-9a0a-561e17376ad4"
-					(reference "#PWR09")
+					(reference "#PWR059")
 					(unit 1)
 				)
@@
 		(dnp no)
 		(fields_autoplaced yes)
-		(property "Reference" "#PWR011"
+		(property "Reference" "#PWR061"
 			(at 219.71 119.38 0)
 			(effects
@@
 			(project "Yet-Another-Nixie-Clock"
 				(path "/78ce616d-4594-460a-a6b5-d8dd90d9a741/3fd9b30e-c53f-44d4-9eb4-8fd367607a00/50401da1-09e6-4577-9a0a-561e17376ad4"
-					(reference "#PWR011")
+					(reference "#PWR061")
 					(unit 1)
 				)
@@
 		(dnp no)
 		(fields_autoplaced yes)
-		(property "Reference" "U1"
+		(property "Reference" "U6"
 			(at 122.7933 81.28 0)
 			(effects
@@
 			(project "Yet-Another-Nixie-Clock"
 				(path "/78ce616d-4594-460a-a6b5-d8dd90d9a741/3fd9b30e-c53f-44d4-9eb4-8fd367607a00/50401da1-09e6-4577-9a0a-561e17376ad4"
-					(reference "U1")
+					(reference "U6")
 					(unit 1)
 				)
@@
 		(dnp no)
 		(fields_autoplaced yes)
-		(property "Reference" "Q2"
+		(property "Reference" "Q3"
 			(at 165.1 87.6299 0)
 			(effects
@@
 			(project "Yet-Another-Nixie-Clock"
 				(path "/78ce616d-4594-460a-a6b5-d8dd90d9a741/3fd9b30e-c53f-44d4-9eb4-8fd367607a00/50401da1-09e6-4577-9a0a-561e17376ad4"
-					(reference "Q2")
+					(reference "Q3")
 					(unit 1)
 				)
@@
 		(dnp no)
 		(fields_autoplaced yes)
-		(property "Reference" "#PWR07"
+		(property "Reference" "#PWR057"
 			(at 120.65 119.38 0)
 			(effects
@@
 			(project "Yet-Another-Nixie-Clock"
 				(path "/78ce616d-4594-460a-a6b5-d8dd90d9a741/3fd9b30e-c53f-44d4-9eb4-8fd367607a00/50401da1-09e6-4577-9a0a-561e17376ad4"
-					(reference "#PWR07")
+					(reference "#PWR057")
 					(unit 1)
 				)
@@
 		(dnp no)
 		(fields_autoplaced yes)
-		(property "Reference" "L1"
+		(property "Reference" "L2"
 			(at 143.51 73.66 90)
 			(effects
@@
 			(project "Yet-Another-Nixie-Clock"
 				(path "/78ce616d-4594-460a-a6b5-d8dd90d9a741/3fd9b30e-c53f-44d4-9eb4-8fd367607a00/50401da1-09e6-4577-9a0a-561e17376ad4"
-					(reference "L1")
+					(reference "L2")
 					(unit 1)
 				)
@@
 		(on_board yes)
 		(dnp no)
-		(property "Reference" "C1"
+		(property "Reference" "C15"
 			(at 72.39 87.7569 0)
 			(effects
@@
 			(project "Yet-Another-Nixie-Clock"
 				(path "/78ce616d-4594-460a-a6b5-d8dd90d9a741/3fd9b30e-c53f-44d4-9eb4-8fd367607a00/50401da1-09e6-4577-9a0a-561e17376ad4"
-					(reference "C1")
+					(reference "C15")
 					(unit 1)
 				)
@@
 		(on_board yes)
 		(dnp no)
-		(property "Reference" "C4"
+		(property "Reference" "C18"
 			(at 186.69 87.7569 0)
 			(effects
@@
 			(project "Yet-Another-Nixie-Clock"
 				(path "/78ce616d-4594-460a-a6b5-d8dd90d9a741/3fd9b30e-c53f-44d4-9eb4-8fd367607a00/50401da1-09e6-4577-9a0a-561e17376ad4"
-					(reference "C4")
+					(reference "C18")
 					(unit 1)
 				)
@@
 		(dnp no)
 		(fields_autoplaced yes)
-		(property "Reference" "#PWR02"
+		(property "Reference" "#PWR052"
 			(at 54.61 81.28 0)
 			(effects
@@
 			(project "Yet-Another-Nixie-Clock"
 				(path "/78ce616d-4594-460a-a6b5-d8dd90d9a741/3fd9b30e-c53f-44d4-9eb4-8fd367607a00/50401da1-09e6-4577-9a0a-561e17376ad4"
-					(reference "#PWR02")
+					(reference "#PWR052")
 					(unit 1)
 				)
@@
 		(dnp no)
 		(fields_autoplaced yes)
-		(property "Reference" "#PWR012"
+		(property "Reference" "#PWR062"
 			(at 236.22 81.28 0)
 			(effects
@@
 			(project "Yet-Another-Nixie-Clock"
 				(path "/78ce616d-4594-460a-a6b5-d8dd90d9a741/3fd9b30e-c53f-44d4-9eb4-8fd367607a00/50401da1-09e6-4577-9a0a-561e17376ad4"
-					(reference "#PWR012")
+					(reference "#PWR062")
 					(unit 1)
 				)
@@
 		(dnp no)
 		(fields_autoplaced yes)
-		(property "Reference" "#PWR06"
+		(property "Reference" "#PWR056"
 			(at 104.14 119.38 0)
 			(effects
@@
 			(project "Yet-Another-Nixie-Clock"
 				(path "/78ce616d-4594-460a-a6b5-d8dd90d9a741/3fd9b30e-c53f-44d4-9eb4-8fd367607a00/50401da1-09e6-4577-9a0a-561e17376ad4"
-					(reference "#PWR06")
+					(reference "#PWR056")
 					(unit 1)
 				)
@@
 		(dnp no)
 		(fields_autoplaced yes)
-		(property "Reference" "R4"
+		(property "Reference" "R20"
 			(at 207.01 107.9499 0)
 			(effects
@@
 			(project "Yet-Another-Nixie-Clock"
 				(path "/78ce616d-4594-460a-a6b5-d8dd90d9a741/3fd9b30e-c53f-44d4-9eb4-8fd367607a00/50401da1-09e6-4577-9a0a-561e17376ad4"
-					(reference "R4")
+					(reference "R20")
 					(unit 1)
 				)
@@
 		(on_board yes)
 		(dnp no)
-		(property "Reference" "C5"
+		(property "Reference" "C19"
 			(at 222.25 87.6362 0)
 			(effects
@@
 			(project "Yet-Another-Nixie-Clock"
 				(path "/78ce616d-4594-460a-a6b5-d8dd90d9a741/3fd9b30e-c53f-44d4-9eb4-8fd367607a00/50401da1-09e6-4577-9a0a-561e17376ad4"
-					(reference "C5")
+					(reference "C19")
 					(unit 1)
 				)
@@
 		(dnp no)
 		(fields_autoplaced yes)
-		(property "Reference" "#PWR04"
+		(property "Reference" "#PWR054"
 			(at 83.82 119.38 0)
 			(effects
@@
 			(project "Yet-Another-Nixie-Clock"
 				(path "/78ce616d-4594-460a-a6b5-d8dd90d9a741/3fd9b30e-c53f-44d4-9eb4-8fd367607a00/50401da1-09e6-4577-9a0a-561e17376ad4"
-					(reference "#PWR04")
+					(reference "#PWR054")
 					(unit 1)
 				)
@@
 		(dnp no)
 		(fields_autoplaced yes)
-		(property "Reference" "#PWR010"
+		(property "Reference" "#PWR060"
 			(at 204.47 119.38 0)
 			(effects
@@
 			(project "Yet-Another-Nixie-Clock"
 				(path "/78ce616d-4594-460a-a6b5-d8dd90d9a741/3fd9b30e-c53f-44d4-9eb4-8fd367607a00/50401da1-09e6-4577-9a0a-561e17376ad4"
-					(reference "#PWR010")
+					(reference "#PWR060")
 					(unit 1)
 				)
@@
 		(dnp no)
 		(fields_autoplaced yes)
-		(property "Reference" "#PWR08"
+		(property "Reference" "#PWR058"
 			(at 161.29 119.38 0)
 			(effects
@@
 			(project "Yet-Another-Nixie-Clock"
 				(path "/78ce616d-4594-460a-a6b5-d8dd90d9a741/3fd9b30e-c53f-44d4-9eb4-8fd367607a00/50401da1-09e6-4577-9a0a-561e17376ad4"
-					(reference "#PWR08")
+					(reference "#PWR058")
 					(unit 1)
 				)
@@
 		(dnp no)
 		(fields_autoplaced yes)
-		(property "Reference" "#PWR03"
+		(property "Reference" "#PWR053"
 			(at 69.85 119.38 0)
 			(effects
@@
 			(project "Yet-Another-Nixie-Clock"
 				(path "/78ce616d-4594-460a-a6b5-d8dd90d9a741/3fd9b30e-c53f-44d4-9eb4-8fd367607a00/50401da1-09e6-4577-9a0a-561e17376ad4"
-					(reference "#PWR03")
+					(reference "#PWR053")
 					(unit 1)
 				)
@@
 		(dnp no)
 		(fields_autoplaced yes)
-		(property "Reference" "#PWR05"
+		(property "Reference" "#PWR055"
 			(at 97.79 119.38 0)
 			(effects
@@
 			(project "Yet-Another-Nixie-Clock"
 				(path "/78ce616d-4594-460a-a6b5-d8dd90d9a741/3fd9b30e-c53f-44d4-9eb4-8fd367607a00/50401da1-09e6-4577-9a0a-561e17376ad4"
-					(reference "#PWR05")
+					(reference "#PWR055")
 					(unit 1)
 				)
@@
 		(on_board yes)
 		(dnp no)
-		(property "Reference" "C2"
+		(property "Reference" "C16"
 			(at 86.36 87.6362 0)
 			(effects
@@
 			(project "Yet-Another-Nixie-Clock"
 				(path "/78ce616d-4594-460a-a6b5-d8dd90d9a741/3fd9b30e-c53f-44d4-9eb4-8fd367607a00/50401da1-09e6-4577-9a0a-561e17376ad4"
-					(reference "C2")
+					(reference "C16")
 					(unit 1)
 				)
@@
 		(dnp no)
 		(fields_autoplaced yes)
-		(property "Reference" "R3"
+		(property "Reference" "R19"
 			(at 207.01 88.8999 0)
 			(effects
@@
 			(project "Yet-Another-Nixie-Clock"
 				(path "/78ce616d-4594-460a-a6b5-d8dd90d9a741/3fd9b30e-c53f-44d4-9eb4-8fd367607a00/50401da1-09e6-4577-9a0a-561e17376ad4"
-					(reference "R3")
+					(reference "R19")
 					(unit 1)
 				)
@@
 		(dnp no)
 		(fields_autoplaced yes)
-		(property "Reference" "D1"
+		(property "Reference" "D3"
 			(at 172.72 72.39 0)
 			(effects
@@
 			(project "Yet-Another-Nixie-Clock"
 				(path "/78ce616d-4594-460a-a6b5-d8dd90d9a741/3fd9b30e-c53f-44d4-9eb4-8fd367607a00/50401da1-09e6-4577-9a0a-561e17376ad4"
-					(reference "D1")
+					(reference "D3")
 					(unit 1)
 				)
@@
 		(on_board yes)
 		(dnp no)
-		(property "Reference" "C3"
+		(property "Reference" "C17"
 			(at 106.68 104.1462 0)
 			(effects
@@
 			(project "Yet-Another-Nixie-Clock"
 				(path "/78ce616d-4594-460a-a6b5-d8dd90d9a741/3fd9b30e-c53f-44d4-9eb4-8fd367607a00/50401da1-09e6-4577-9a0a-561e17376ad4"
-					(reference "C3")
-					(unit 1)
-				)
+					(reference "C17")
+					(unit 1)
+				)
