File: Hardware/Yet-Another-Nixie-Clock/sch/nixie.kicad_sch (KiCad schematic)
At the start: 13 parts, among them J2 Nixie IN12, Q1 BF820, Q10 BF820, Q11 BF820, Q3 BF820, Q4 BF820, Q5 BF820, Q6 BF820, Q7 BF820, Q72 PMBTA92, Q8 BF820, Q9 BF820

Commit message: Schematic work
Parts:
- removed Q1, Q10, Q11, Q3, Q4, Q5, Q6, Q7, Q8, Q9: BF820, Package_TO_SOT_SMD:TSOT-23, symbol Transistor_BJT:Q_NPN_BCE
- renumbered Q72 to Q14, R1 to R10
Connections:
- net ANODE renamed A

Commit message: Schematic work
Parts:
- added Q20: PMBTA42, Package_TO_SOT_SMD:SOT-23, symbol Transistor_BJT:MMBT2222A
- added R23: 300k, symbol Device:R_Small_US
- added R29, R35: 4.7k, symbol Device:R_Small_US
- R10: value R_Small_US -> 10k
Connections:
- net A: now also R29.2
- net G_A: now also R35.2
- net at Q14.1 (B): now also R10.2, R23.1
- net at Q14.2 (C): now also R29.1
- net VCCHV: now reaches Q14.3 (E), R10.1
- new net: Q20.1 (B), R35.1
- new net: Q20.3 (C), R23.2
- new net GND: Q20.2 (E)
- no-connect marks 0 -> 1
Other:
- moved on the sheet: J2, Q14, R10

Commit message: Schematic work and fixes
Parts:
- J2: now left out of the parts list
- Q14: footprint (none) -> Package_TO_SOT_SMD:TSOT-23; symbol Transistor_BJT:Q_PNP_BCE -> Transistor_BJT:Q_PNP_BEC; LCSC (none) -> C282560
- Q20: symbol Transistor_BJT:MMBT2222A -> Transistor_BJT:Q_PNP_BEC
Connections:
- net VCCHV: now also Q14.2 (E); no longer Q14.3 (E)
- net at R29.1: now also Q14.3 (C); no longer Q14.2 (C)
Changed lines of the file:
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@@
 	)
 	(symbol
-		(lib_id "Transistor_BJT:Q_PNP_BCE")
+		(lib_id "Transistor_BJT:Q_PNP_BEC")
 		(at 132.08 120.65 0)
 		(mirror x)
@@
 			)
 		)
-		(property "Footprint" ""
+		(property "Footprint" "Package_TO_SOT_SMD:TSOT-23"
 			(at 137.16 123.19 0)
 			(effects
@@
 			)
 		)
-		(property "Description" "PNP transistor, base/collector/emitter"
+		(property "Description" "PNP transistor, base/emitter/collector"
+			(at 132.08 120.65 0)
+			(effects
+				(font
+					(size 1.27 1.27)
+				)
+				(hide yes)
+			)
+		)
+		(property "LCSC" "C282560"
 			(at 132.08 120.65 0)
 			(effects
@@
 	)
 	(symbol
-		(lib_id "Transistor_BJT:MMBT2222A")
+		(lib_id "Transistor_BJT:Q_PNP_BEC")
 		(at 110.49 127 0)
 		(unit 1)
@@
 		)
 		(property "Footprint" "Package_TO_SOT_SMD:SOT-23"
-			(at 115.57 128.905 0)
-			(effects
-				(font
-					(size 1.27 1.27)
-					(italic yes)
-				)
-				(justify left)
-				(hide yes)
-			)
-		)
-		(property "Datasheet" "https://assets.nexperia.com/documents/data-sheet/MMBT2222A.pdf"
+			(at 115.57 124.46 0)
+			(effects
+				(font
+					(size 1.27 1.27)
+				)
+				(hide yes)
+			)
+		)
+		(property "Datasheet" "~"
 			(at 110.49 127 0)
 			(effects
@@
 					(size 1.27 1.27)
 				)
-				(justify left)
-				(hide yes)
-			)
-		)
-		(property "Description" "600mA Ic, 40V Vce, NPN Transistor, SOT-23"
+				(hide yes)
+			)
+		)
+		(property "Description" "PNP transistor, base/emitter/collector"
 			(at 110.49 127 0)
 			(effects
@@
 		(unit 1)
 		(exclude_from_sim no)
-		(in_bom yes)
-		(on_board yes)
-		(dnp no)
+		(in_bom no)
+		(on_board yes)
+		(dnp no)

Commit message: Schematic work and fixes
Parts:
- renumbered J2 to J4, Q20 to Q4, Q14 to Q5, R35 to R21, R23 to R22, R10 to R23, R29 to R24
