File: Hardware/Yet-Another-Nixie-Clock/sch/nixie_driver.kicad_sch (KiCad schematic)
At the start: 1 part

Commit message: Schematic work
Parts:
- added D10, D11, D12, D4, D5, D6, D7, D8, D9: BAV103, Diode_SMD:D_MiniMELF, symbol Device:D_Small
- added Q10, Q11, Q12, Q13, Q4, Q5, Q6, Q7, Q8, Q9: BF820, Package_TO_SOT_SMD:TSOT-23, symbol Transistor_BJT:Q_NPN_BCE
- added U15, U17: 74HC237, symbol 74xx:74HC237
Connections:
- net at D3.1 (K): now also D10.1 (K), D11.1 (K), D12.1 (K), D4.1 (K), D5.1 (K), D6.1 (K), D7.1 (K), D8.1 (K), D9.1 (K)
- net K0: now reaches D3.2 (A)
- net K0: now also Q4.2 (C)
- new net GND: Q10.3 (E), Q11.3 (E), Q12.3 (E), Q13.3 (E), Q4.3 (E), Q5.3 (E), Q6.3 (E), Q7.3 (E), Q8.3 (E), Q9.3 (E)
- new net G_K0: Q4.1 (B), U17.15 (Y0)
- new net G_K1: Q5.1 (B), U17.14 (Y1)
- new net G_K2: Q6.1 (B), U17.13 (Y2)
- new net G_K3: Q7.1 (B), U17.12 (Y3)
- new net G_K4: Q8.1 (B), U17.11 (Y4)
- new net G_K5: Q9.1 (B), U17.10 (Y5)
- new net G_K6: Q10.1 (B), U17.9 (Y6)
- new net G_K7: Q11.1 (B), U17.7 (Y7)
- new net G_K8: Q12.1 (B), U15.15 (Y0)
- new net G_K9: Q13.1 (B), U15.14 (Y1)
- new net K1: D4.2 (A), Q5.2 (C)
- new net K2: D5.2 (A), Q6.2 (C)
- new net K3: D6.2 (A), Q7.2 (C)
- new net K4: D7.2 (A), Q8.2 (C)
- new net K5: D8.2 (A), Q9.2 (C)
- new net K6: D9.2 (A), Q10.2 (C)
- new net K7: D10.2 (A), Q11.2 (C)
- new net K8: D11.2 (A), Q12.2 (C)
- new net K9: D12.2 (A), Q13.2 (C)
- new net N0: U15.1 (A0), U17.1 (A0)
- new net N1: U15.2 (A1), U17.2 (A1)
- new net N2: U15.3 (A2), U17.3 (A2)
- new net N3: U15.6 (E2), U17.5 (~{E1})
- new net ~{N_LE}: U15.4 (~{LE}), U17.4 (~{LE})
- no-connect marks 0 -> 6
Other:
- removed sheet Nixie6
- removed sheet Shift Register0
- removed sheet Shift Register1
- removed sheet Shift Register2
- removed sheet Shift Register3
- removed sheet Shift Register4
- removed sheet Shift Register5
- removed sheet Shift Register6
- removed sheet Shift Register7
- sheet Nixie0: file sch/nixie.kicad_sch -> nixie.kicad_sch
- sheet Nixie0 ports: added G_A, K[0..9]; removed ANODE, CATHODE_GATES[0..9]
- sheet Nixie1: file sch/nixie.kicad_sch -> nixie.kicad_sch
- sheet Nixie1 ports: added G_A, K[0..9]; removed ANODE, CATHODE_GATES[0..9]
- sheet Nixie2: file sch/nixie.kicad_sch -> nixie.kicad_sch
- sheet Nixie2 ports: added G_A, K[0..9]; removed ANODE, CATHODE_GATES[0..9]
- sheet Nixie3: file sch/nixie.kicad_sch -> nixie.kicad_sch
- sheet Nixie3 ports: added G_A, K[0..9]; removed ANODE, CATHODE_GATES[0..9]
- sheet Nixie4: file sch/nixie.kicad_sch -> nixie.kicad_sch
- sheet Nixie4 ports: added G_A, K[0..9]; removed ANODE, CATHODE_GATES[0..9]
- sheet Nixie5: file sch/nixie.kicad_sch -> nixie.kicad_sch
- sheet Nixie5 ports: added G_A, K[0..9]; removed ANODE, CATHODE_GATES[0..9]
- moved on the sheet: D3

Commit message: Schematic work
Parts:
- added C20, C21: 100nF, Capacitor_SMD:C_0603_1608Metric, symbol Device:C_Small
- added D13: 100V, Diode_SMD:D_SMA, symbol Device:D_Zener_Small
- U15, U17: LCSC (none) -> C2674656
Connections:
- net GND: now also U15.5 (~{E1}), U15.8 (GND), U17.8 (GND), C20.1, C21.1, D13.2 (A)
- net at D10.1 (K), D11.1 (K), D12.1 (K)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: now also D13.1 (K)
- net VCC3V3: now reaches U17.16 (VCC)
- net VCC3V3: now also U15.16 (VCC), U17.6 (E2), C20.2, C21.2
Other:
- added sheet HV PSU (sch/hv_psu.kicad_sch)
- moved on the sheet: D10, D11, D12, D3, D4, D5, D6, D7, D8, D9, Q4, Q5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

Commit message: Schematic work and fixes
Parts:
- added R41, R42: 10k, symbol Device:R_Small_US
- added RN1: R_Pack08_Split, symbol Device:R_Pack08_Split
- Q10, Q11, Q12, Q13, Q4, Q5, Q6, Q7, Q8, Q9: symbol Transistor_BJT:Q_NPN_BCE -> Transistor_BJT:Q_NPN_BEC
Connections:
- net GND: now also Q10.2 (E), Q11.2 (E), Q12.2 (E), Q13.2 (E), Q4.2 (E), Q5.2 (E), Q6.2 (E), Q7.2 (E), Q8.2 (E), Q9.2 (E); no longer Q10.3 (E), Q11.3 (E), Q12.3 (E), Q13.3 (E), Q4.3 (E), Q5.3 (E), Q6.3 (E), Q7.3 (E), Q8.3 (E), Q9.3 (E)
- net G_K0: now also RN1.1 (R1.1); no longer Q4.1 (B)
- net G_K1: now also RN1.2 (R2.1); no longer Q5.1 (B)
- net G_K2: now also RN1.3 (R3.1); no longer Q6.1 (B)
- net G_K3: now also RN1.4 (R4.1); no longer Q7.1 (B)
- net G_K4: now also RN1.5 (R5.1); no longer Q8.1 (B)
- net G_K5: now also RN1.6 (R6.1); no longer Q9.1 (B)
- net G_K6: now also RN1.7 (R7.1); no longer Q10.1 (B)
- net G_K7: now also RN1.8 (R8.1); no longer Q11.1 (B)
- net G_K8: now also R41.1; no longer Q12.1 (B)
- net G_K9: now also R42.1; no longer Q13.1 (B)
- net K0: now also Q4.3 (C); no longer Q4.2 (C)
- net K1: now also Q5.3 (C); no longer Q5.2 (C)
- net K2: now also Q6.3 (C); no longer Q6.2 (C)
- net K3: now also Q7.3 (C); no longer Q7.2 (C)
- net K4: now also Q8.3 (C); no longer Q8.2 (C)
- net K5: now also Q9.3 (C); no longer Q9.2 (C)
- net K6: now also Q10.3 (C); no longer Q10.2 (C)
- net K7: now also Q11.3 (C); no longer Q11.2 (C)
- net K8: now also Q12.3 (C); no longer Q12.2 (C)
- net K9: now also Q13.3 (C); no longer Q13.2 (C)
- new net: Q11.1 (B), RN1.9 (R8.2)
- new net: Q5.1 (B), RN1.15 (R2.2)
- new net: Q12.1 (B), R41.2
- new net: Q7.1 (B), RN1.13 (R4.2)
- new net: Q4.1 (B), RN1.16 (R1.2)
- new net: Q6.1 (B), RN1.14 (R3.2)
- new net: Q8.1 (B), RN1.12 (R5.2)
- new net: Q9.1 (B), RN1.11 (R6.2)
- new net: Q13.1 (B), R42.2
- new net: Q10.1 (B), RN1.10 (R7.2)

Commit message: Schematic work and fixes
Parts:
- renumbered D9 to D10, D10 to D11, D11 to D12, D12 to D13, D13 to D14, D3 to D4, D4 to D5, D5 to D6, D6 to D7, D7 to D8, D8 to D9, Q8 to Q10, Q9 to Q11, Q10 to Q12, Q11 to Q13, Q12 to Q14, Q13 to Q15, Q4 to Q6, Q5 to Q7, Q6 to Q8, Q7 to Q9, R41 to R25, R42 to R26, U17 to U7, U15 to U8
Other:
- sheet HV PSU: file sch/hv_psu.kicad_sch -> hv_psu.kicad_sch
