File: Hardware/Yet-Another-Nixie-Clock-Face/Yet-Another-Nixie-Clock-Face.kicad_pcb (KiCad board)
At the start: 4 copper layers, 200 x 70 mm, 79 parts, among them J10 Conn_02x06_Odd_Even, J11 Conn_02x06_Odd_Even, J4 Nixie IN12, J5 Nixie IN12, J6 Nixie IN12, J7 Nixie IN12, J8 Nixie IN12, J9 Nixie IN12, Q10 BF820, Q11 BF820, Q12 BF820, Q13 BF820, Q14 BF820, Q15 BF820, Q16 PMBTA42, Q17 PMBTA92, Q18 PMBTA42, Q19 PMBTA92, Q20 PMBTA42, Q21 PMBTA92, Q22 PMBTA42, Q23 PMBTA92, Q24 PMBTA42, Q25 PMBTA92, Q4 PMBTA42, Q5 PMBTA92, Q6 BF820, Q7 BF820, Q8 BF820, Q9 BF820, U7 74HC237, U8 74HC237

Commit message: Minor improvements
Parts:
- R1: moved to B.Cu
- moved D1 138.0 mm to (121.6, 100.2), turned to -45 degrees
- moved D2 79.8 mm to (181.6, 100.2), turned to -45 degrees
- moved R1 21.6 mm to (235.5, 119.6)
- moved R23 0.94 mm to (240.0, 103.4)
- moved Q4 0.94 mm to (236.9, 99.5)
- moved Q5 0.94 mm to (236.8, 103.2)
- moved R21 0.94 mm to (233.7, 99.6)
- moved R22 0.94 mm to (240.0, 100.3)
- moved R24 0.94 mm to (233.7, 103.2)
- turned R30 to 180 degrees
Routing:
- net Net-(D1-A): track 0.00 -> 149.2 mm, vias 0 -> 5
- net /G_A0: track 0.00 -> 20.0 mm
- net /Nixie Driver/K2: track 223.4 -> 206.6 mm
- net VCCHV: track 0.00 -> 12.3 mm
- net /Nixie Driver/K1: track 204.7 -> 192.7 mm
- net /Nixie Driver/Nixie4/A: track 4.80 -> 16.5 mm
- net /Nixie Driver/Nixie2/A: track 4.99 -> 15.9 mm
- net /Nixie Driver/Nixie1/A: track 4.71 -> 11.2 mm
- net /Nixie Driver/Nixie5/A: track 4.95 -> 11.2 mm
- net /Nixie Driver/Nixie3/A: track 5.12 -> 11.4 mm
- net /LED: track 0.00 -> 4.71 mm
- net /Nixie Driver/Nixie0/A: track 4.95 -> 9.40 mm
- net GND: track 7.81 -> 12.0 mm, vias 5 -> 7
- net Net-(Q5-B): track 0.00 -> 3.73 mm
- net Net-(Q19-B): track 0.00 -> 3.49 mm
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
Commit message: Major schematic and layout advancements
Parts:
- J4, J5, J6, J7, J8, J9: footprint Yet-Another-Nixie-Clock:IN_12B_Socket -> Yet-Another-Nixie-Clock-Face:IN_12B_Socket
Routing:
- net VCCHV: track 12.3 -> 284.9 mm, vias 0 -> 6
- net VCC3V3: track 87.9 -> 96.4 mm, vias 1 -> 0
- net /Nixie Driver/K2: track 206.6 -> 203.3 mm
- net /Nixie Driver/K0: track 228.6 -> 231.4 mm, vias 6 -> 7
- net GND: track 12.0 -> 10.1 mm, vias 7 -> 66
- net /Nixie Driver/K1: track 192.7 -> 191.3 mm
- added copper zone on B.Cu, net GND
- added copper zone on F.Cu, net GND
- added copper zone on B.Cu, net VCCHV
Other:
- copper layers 4 -> 2
- board text added: "Yet Another Nixie Clock Afonso Muralha 2025"
