File: Hardware/Yet-Another-Nixie-Clock-Face/Yet-Another-Nixie-Clock-Face.kicad_sch (KiCad schematic)
At the start: 9 parts, among them J10 Conn_02x06_Odd_Even, J11 Conn_02x06_Odd_Even

Commit message: Minor touches. Fixed bom. Exported production files
Parts:
- D1, D2: now left out of the parts list
- J10, J11: LCSC (none) -> C3294464
- R1: LCSC (none) -> C22548
Changed lines of the file:
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@@
+			)
+		)
+		(property "LCSC" "C3294464"
+			(at 275.59 138.43 0)
+			(effects
+				(font
+					(size 1.27 1.27)
+				)
+				(hide yes)
 			)
 		)
@@
 			)
 		)
+		(property "LCSC" "C3294464"
+			(at 165.1 135.89 0)
+			(effects
+				(font
+					(size 1.27 1.27)
+				)
+				(hide yes)
+			)
+		)
 		(pin "6"
 		)
@@
 			)
 		)
-		(property "LCSC" ""
+		(property "LCSC" "C22548"
 			(at 275.59 167.64 0)
 			(effects
@@
 		(unit 1)
 		(exclude_from_sim no)
-		(in_bom yes)
+		(in_bom no)
 		(on_board yes)
 		(dnp no)
@@
 		(unit 1)
 		(exclude_from_sim no)
-		(in_bom yes)
-		(on_board yes)
-		(dnp no)
+		(in_bom no)
+		(on_board yes)
+		(dnp no)
