File: Hardware/Yet-Another-Nixie-Clock-Face/sch/nixie.kicad_sch (KiCad schematic)
At the start: 7 parts, among them J4 Nixie IN12, Q4 PMBTA42, Q5 PMBTA92

Commit message: Schematic advancements, separated boards
Parts:
- J4: footprint Yet-Another-Nixie-Clock:IN_12B_Socket -> Yet-Another-Nixie-Clock-Face:IN_12B_Socket
Changed lines of the file:
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@@
 			)
 		)
-		(property "Footprint" "Yet-Another-Nixie-Clock:IN_12B_Socket"
+		(property "Footprint" "Yet-Another-Nixie-Clock-Face:IN_12B_Socket"
 			(at 186.69 76.2 0)
 			(effects

Commit message: Minor touches. Fixed bom. Exported production files
Parts:
- Q4: LCSC (none) -> C417384
- R21, R24: LCSC (none) -> C99782
- R22: LCSC (none) -> C114667
- R23: LCSC (none) -> C98220
Changed lines of the file:
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@@
+			)
+		)
+		(property "LCSC" "C99782"
+			(at 99.06 127 90)
+			(effects
+				(font
+					(size 1.27 1.27)
+				)
+				(hide yes)
 			)
 		)
@@
 			)
 		)
+		(property "LCSC" "C417384"
+			(at 110.49 127 0)
+			(effects
+				(font
+					(size 1.27 1.27)
+				)
+				(hide yes)
+			)
+		)
 		(pin "2"
 		)
@@
 		(property "Description" "Resistor, small US symbol"
 			(at 116.84 120.65 0)
+			(effects
+				(font
+					(size 1.27 1.27)
+				)
+				(hide yes)
+			)
+		)
+		(property "LCSC" "C114667"
+			(at 116.84 120.65 90)
 			(effects
 				(font
@@
 			)
 		)
+		(property "LCSC" "C99782"
+			(at 134.62 129.54 0)
+			(effects
+				(font
+					(size 1.27 1.27)
+				)
+				(hide yes)
+			)
+		)
 		(pin "1"
 		)
@@
 			(at 123.19 116.84 0)
 			(effects
+				(font
+					(size 1.27 1.27)
+				)
+				(hide yes)
+			)
+		)
+		(property "LCSC" "C98220"
+			(at 123.19 116.84 0)
+			(effects
