File: Hardware/Yet-Another-Nixie-Clock-Face/sch/nixie_driver.kicad_sch (KiCad schematic)
At the start: 28 parts, among them Q10 BF820, Q11 BF820, Q12 BF820, Q13 BF820, Q14 BF820, Q15 BF820, Q6 BF820, Q7 BF820, Q8 BF820, Q9 BF820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

Commit message: Schematic advancements, separated boards
Other:
- removed sheet HV PSU
Changed lines of the file:
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@@
 		)
 		(instances
-			(project "Yet-Another-Nixie-Clock"
+			(project "Yet-Another-Nixie-Clock-Face"
 				(path "/78ce616d-4594-460a-a6b5-d8dd90d9a741/3fd9b30e-c53f-44d4-9eb4-8fd367607a00"
 					(page "5")
@@
 		)
 		(instances
-			(project "Yet-Another-Nixie-Clock"
+			(project "Yet-Another-Nixie-Clock-Face"
 				(path "/78ce616d-4594-460a-a6b5-d8dd90d9a741/3fd9b30e-c53f-44d4-9eb4-8fd367607a00"
 					(page "9")
@@
 		)
 		(instances
-			(project "Yet-Another-Nixie-Clock"
+			(project "Yet-Another-Nixie-Clock-Face"
 				(path "/78ce616d-4594-460a-a6b5-d8dd90d9a741/3fd9b30e-c53f-44d4-9eb4-8fd367607a00"
 					(page "3")
-				)
-			)
-		)
-	)
-	(sheet
-		(at 44.45 26.67)
-		(size 43.18 17.78)
-		(exclude_from_sim no)
-		(in_bom yes)
-		(on_board yes)
-		(dnp no)
-		(fields_autoplaced yes)
-		(stroke
-			(width 0.1524)
-			(type solid)
-		)
-		(fill
-			(color 0 0 0 0.0000)
-		)
-		(property "Sheetname" "HV PSU"
-			(at 44.45 25.9584 0)
-			(effects
-				(font
-					(size 1.27 1.27)
-				)
-				(justify left bottom)
-			)
-		)
-		(property "Sheetfile" "hv_psu.kicad_sch"
-			(at 44.45 45.0346 0)
-			(effects
-				(font
-					(size 1.27 1.27)
-				)
-				(justify left top)
-			)
-		)
-		(instances
-			(project "Yet-Another-Nixie-Clock"
-				(path "/78ce616d-4594-460a-a6b5-d8dd90d9a741/3fd9b30e-c53f-44d4-9eb4-8fd367607a00"
-					(page "2")
 				)
 			)
@@
 		)
 		(instances
-			(project "Yet-Another-Nixie-Clock"
+			(project "Yet-Another-Nixie-Clock-Face"
 				(path "/78ce616d-4594-460a-a6b5-d8dd90d9a741/3fd9b30e-c53f-44d4-9eb4-8fd367607a00"
 					(page "8")
@@
 		)
 		(instances
-			(project "Yet-Another-Nixie-Clock"
+			(project "Yet-Another-Nixie-Clock-Face"
 				(path "/78ce616d-4594-460a-a6b5-d8dd90d9a741/3fd9b30e-c53f-44d4-9eb4-8fd367607a00"
 					(page "7")
@@
 		)
 		(instances
-			(project "Yet-Another-Nixie-Clock"
+			(project "Yet-Another-Nixie-Clock-Face"
 				(path "/78ce616d-4594-460a-a6b5-d8dd90d9a741/3fd9b30e-c53f-44d4-9eb4-8fd367607a00"
 					(page "6")

Commit message: Minor touches. Fixed bom. Exported production files
Parts:
- RN1: LCSC (none) -> C326649
Changed lines of the file:
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@@
 			)
 		)
+		(property "LCSC" "C326649"
+			(at 194.31 87.63 90)
+			(effects
+				(font
+					(size 1.27 1.27)
+				)
+				(hide yes)
+			)
+		)
 		(pin "8"
 		)
@@
 			)
 		)
+		(property "LCSC" "C326649"
+			(at 138.43 64.77 90)
+			(effects
+				(font
+					(size 1.27 1.27)
+				)
+				(hide yes)
+			)
+		)
 		(pin "8"
 		)
@@
 			)
 		)
+		(property "LCSC" "C326649"
+			(at 139.7 134.62 90)
+			(effects
+				(font
+					(size 1.27 1.27)
+				)
+				(hide yes)
+			)
+		)
 		(pin "8"
 		)
@@
 			)
 		)
+		(property "LCSC" "C326649"
+			(at 139.7 110.49 90)
+			(effects
+				(font
+					(size 1.27 1.27)
+				)
+				(hide yes)
+			)
+		)
 		(pin "8"
 		)
@@
 			)
 		)
+		(property "LCSC" "C326649"
+			(at 138.43 43.18 90)
+			(effects
+				(font
+					(size 1.27 1.27)
+				)
+				(hide yes)
+			)
+		)
 		(pin "8"
 		)
@@
 			)
 		)
+		(property "LCSC" "C326649"
+			(at 139.7 87.63 90)
+			(effects
+				(font
+					(size 1.27 1.27)
+				)
+				(hide yes)
+			)
+		)
 		(pin "8"
 		)
@@
 			)
 		)
+		(property "LCSC" "C326649"
+			(at 194.31 43.18 90)
+			(effects
+				(font
+					(size 1.27 1.27)
+				)
+				(hide yes)
+			)
+		)
 		(pin "8"
 		)
@@
 			(effects
 				(font
+					(size 1.27 1.27)
+				)
+				(hide yes)
+			)
+		)
+		(property "LCSC" "C326649"
+			(at 194.31 64.77 90)
+			(effects
+				(font
