File: Hardware/Yet-Another-Nixie-Clock-Processing/Yet-Another-Nixie-Clock-Processing.kicad_pcb (KiCad board)
At the start: 4 copper layers, 200 x 70 mm, 56 parts, among them J1 PJ-002BH, J10 Conn_02x06_Odd_Even, J11 Conn_02x06_Odd_Even, J2 USB_C_Receptacle_USB2.0, Q1 MMBT2222A, Q2 MMBT2222A, Q3 Q_NMOS, SW1 SW_MEC_5E, SW2 SW_MEC_5E, SW3 SW_MEC_5E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

Commit message: Major schematic and layout advancements
Parts:
- removed D1: Green, LED_SMD:LED_0603_1608Metric
- removed D15: LED, LED_SMD:LED_0603_1608Metric
- removed H1, H4: MountingHole_Pad, MountingHole:MountingHole_3.2mm_M3_Pad
- removed R16: 0, Resistor_SMD:R_0402_1005Metric
- added BT1: Battery_Cell, Yet-Another-Nixie-Clock-Face:BAT-TH_CR2032-BS-6-1, B.Cu at (218.3, 116.3)
- added D4: LED, LED_SMD:LED_0603_1608Metric, B.Cu at (249.3, 90.4)
- added J3: JTAG, Connector_IDC:IDC-Header_2x05_P2.54mm_Vertical, B.Cu at (223.5, 71.7)
- added R1: 10k, Resistor_SMD:R_0603_1608Metric, F.Cu at (221.0, 96.4)
- added R10: 1k, Resistor_SMD:R_0603_1608Metric, F.Cu at (243.0, 90.4)
- added R11: 1k, Resistor_SMD:R_0603_1608Metric, F.Cu at (239.8, 90.4)
- added R12: 10k, Resistor_SMD:R_0603_1608Metric, B.Cu at (243.7, 111.1)
- added R13: 10k, Resistor_SMD:R_0603_1608Metric, B.Cu at (248.4, 111.0)
- added R17: 10k, Resistor_SMD:R_0603_1608Metric, B.Cu at (239.3, 111.1)
- added R2: 10k, Resistor_SMD:R_0603_1608Metric, F.Cu at (222.7, 96.4)
- added R21: 1k, Resistor_SMD:R_0603_1608Metric, F.Cu at (249.3, 90.4)
- added R3: 10k, Resistor_SMD:R_0603_1608Metric, F.Cu at (234.6, 94.5)
- added R6: 33.2k, Resistor_SMD:R_0603_1608Metric, F.Cu at (226.3, 88.1)
- added R7: 10k, Resistor_SMD:R_0603_1608Metric, F.Cu at (229.5, 88.1)
- added R9: 1k, Resistor_SMD:R_0603_1608Metric, F.Cu at (246.2, 90.4)
- C5, D16, D17, D2, R4, R5, U3: moved to B.Cu
- J1, J10, J11, U5: moved to F.Cu
- R14, R15: footprint Resistor_SMD:R_0402_1005Metric -> Resistor_SMD:R_0603_1608Metric
- SW1, SW2, SW3: footprint Yet-Another-Nixie-Clock-Processing:SW_SKRPACE010 -> Yet-Another-Nixie-Clock:SW_SKRPACE010; moved to B.Cu
- moved C5 206.6 mm to (237.6, 94.7), turned to 180 degrees
- moved C1 203.2 mm to (234.7, 87.2), turned to -90 degrees
- moved C2 202.4 mm to (233.1, 87.2), turned to -90 degrees
- moved C3 202.1 mm to (229.3, 80.0), turned to 180 degrees
- moved C4 197.4 mm to (228.1, 92.8)
- moved C8 197.0 mm to (233.0, 94.5), turned to 90 degrees
- moved C7 194.8 mm to (231.5, 94.5), turned to -90 degrees
- moved C6 191.8 mm to (228.1, 91.3), turned to 180 degrees
- moved C10 190.3 mm to (221.9, 88.2), turned to 180 degrees
- moved C9 188.9 mm to (222.0, 89.8), turned to 180 degrees
- moved C11 186.8 mm to (226.3, 89.7)
- moved C14 184.2 mm to (226.0, 105.0)
- moved C13 180.6 mm to (226.3, 119.4), turned to 180 degrees
- moved U4 176.1 mm to (228.7, 112.0), turned to 90 degrees
- moved C12 171.1 mm to (209.6, 91.8), turned to 180 degrees
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Connections:
- D2 pad 1: GND -> Net-(D2-K)
- J10 pad 1: /G_A0 -> /G_A5
- J10 pad 10: /N3 -> /G_A4
- J10 pad 11: /~{N_LE} -> /LED_1
- J10 pad 12: GND -> /~{N_LE}
- J10 pad 2: /G_A5 -> /G_A0
- J10 pad 3: /G_A1 -> /N0
- J10 pad 4: /N0 -> /G_A1
- J10 pad 5: /G_A2 -> /N1
- J10 pad 6: /N1 -> /G_A2
- J10 pad 7: /G_A3 -> /N2
- J10 pad 8: /N2 -> /G_A3
- J10 pad 9: /G_A4 -> /N3
- J11 pad 7: unconnected-(J11-Pin_7-Pad7) -> VCC3V3
- J11 pad 8: unconnected-(J11-Pin_8-Pad8) -> VCC3V3
- U1 pad 13: unconnected-(U1-~{RXT}/GPIO.1-Pad13) -> Net-(D4-K)
- U1 pad 14: unconnected-(U1-~{TXT}/GPIO.0-Pad14) -> Net-(D2-K)
- U5 pad 10: /G_A0 -> /G_A3
- U5 pad 11: /G_A1 -> /N2
- U5 pad 26: /LED_1 -> /G_A0
- U5 pad 27: /N0 -> /G_A1
- U5 pad 28: /N1 -> /G_A5
- U5 pad 30: /N2 -> /N0
- U5 pad 31: /N3 -> /N1
- U5 pad 6: /G_A5 -> /LED_1
- U5 pad 8: /G_A3 -> /G_A4
- U5 pad 9: /G_A4 -> /N3
Routing:
- net VCC3V3: track 0.00 -> 138.0 mm, vias 0 -> 8
- net /SW1: track 0.00 -> 72.9 mm, vias 0 -> 3
- net /IO0: track 0.00 -> 67.3 mm, vias 0 -> 2
- net /~{N_LE}: track 0.00 -> 66.8 mm, vias 0 -> 2
- net /G_A4: track 0.00 -> 65.2 mm, vias 0 -> 2
- net /ESP_RST: track 0.00 -> 64.3 mm, vias 0 -> 3
- net /G_A0: track 0.00 -> 60.8 mm, vias 0 -> 2
- net /N1: track 0.00 -> 60.7 mm, vias 0 -> 2
- net /G_A3: track 0.00 -> 60.3 mm, vias 0 -> 2
- net GND: track 0.00 -> 60.2 mm, vias 0 -> 88
- net /G_A1: track 0.00 -> 58.7 mm, vias 0 -> 2
- net /LED_1: track 0.00 -> 58.1 mm, vias 0 -> 2
- net /N0: track 0.00 -> 57.5 mm, vias 0 -> 2
- net /RTC_SDA: track 0.00 -> 56.8 mm, vias 0 -> 3
- net /RTC_SCL: track 0.00 -> 55.9 mm, vias 0 -> 3
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- added copper zone on B.Cu, net GND
- added copper zone on F.Cu, net GND
- added copper zone on In1.Cu, net GND
- added copper zone on In2.Cu, net GND
- added copper zone on F.Cu, net Net-(D3-A)
- added copper zone on F.Cu, net Net-(Q3-G)
- added copper zone on F.Cu, net Net-(Q3-S)
- added copper zone on F.Cu, net Net-(U2-SW)
- added copper zone on F.Cu, net VCC12V
- added copper zone on In2.Cu, net VCC12V
- added copper zone on F.Cu, net VCC3V3
- added copper zone on F.Cu, net VCCHV
Other:
- board size 200 x 70 mm -> 59.7 x 70 mm
- board text added: "BOOT0"
- board text added: "RST"
- board text added: "SW1"
