File: Hardware/Yet-Another-Nixie-Clock-Processing/Yet-Another-Nixie-Clock-Processing.kicad_sch (KiCad schematic)
At the start: 57 parts, among them J1 PJ-002BH, J10 Conn_02x06_Odd_Even, J11 Conn_02x06_Odd_Even, J2 USB_C_Receptacle_USB2.0, J3 JTAG, Q1 MMBT2222A, Q2 MMBT2222A, SW1 SW_MEC_5E, SW2 SW_MEC_5E, SW3 SW_MEC_5E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

Commit message: Schematic advancements, separated boards
Parts:
- SW1, SW2, SW3: footprint Yet-Another-Nixie-Clock:SW_SKRPACE010 -> Yet-Another-Nixie-Clock-Processing:SW_SKRPACE010
Other:
- removed sheet Nixie Driver
- added sheet HV PSU (sch/hv_psu.kicad_sch)
Changed lines of the file:
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@@
 		)
 	)
-	(bus
-		(pts
-			(xy 292.1 157.48) (xy 302.26 157.48)
-		)
-		(stroke
-			(width 0)
-			(type default)
-		)
-	)
 	(wire
 		(pts
@@
 		)
 	)
-	(bus
-		(pts
-			(xy 292.1 160.02) (xy 302.26 160.02)
-		)
-		(stroke
-			(width 0)
-			(type default)
-		)
-	)
 	(wire
 		(pts
@@
 	(wire
 		(pts
-			(xy 292.1 162.56) (xy 302.26 162.56)
-		)
-		(stroke
-			(width 0)
-			(type default)
-		)
-	)
-	(wire
-		(pts
 			(xy 245.11 120.65) (xy 248.92 120.65)
 		)
@@
 		)
 	)
-	(label "~{N_LE}"
-		(at 292.1 162.56 0)
-		(effects
-			(font
-				(size 1.27 1.27)
-			)
-			(justify left bottom)
-		)
-	)
-	(label "G_A[0..5]"
-		(at 292.1 160.02 0)
-		(effects
-			(font
-				(size 1.27 1.27)
-			)
-			(justify left bottom)
-		)
-	)
 	(label "G_A[0..5]"
 		(at 349.25 78.74 180)
@@
 		)
 	)
-	(label "N[0..3]"
-		(at 292.1 157.48 0)
-		(effects
-			(font
-				(size 1.27 1.27)
-			)
-			(justify left bottom)
-		)
-	)
 	(label "LED_3"
 		(at 279.4 120.65 180)
@@
 			)
 		)
-		(property "Footprint" "Yet-Another-Nixie-Clock:SW_SKRPACE010"
+		(property "Footprint" "Yet-Another-Nixie-Clock-Processing:SW_SKRPACE010"
 			(at 358.14 81.28 0)
 			(effects
@@
 			)
 		)
-		(property "Footprint" "Yet-Another-Nixie-Clock:SW_SKRPACE010"
+		(property "Footprint" "Yet-Another-Nixie-Clock-Processing:SW_SKRPACE010"
 			(at 251.46 44.45 0)
 			(effects
@@
 			)
 		)
-		(property "Footprint" "Yet-Another-Nixie-Clock:SW_SKRPACE010"
+		(property "Footprint" "Yet-Another-Nixie-Clock-Processing:SW_SKRPACE010"
 			(at 260.35 78.74 0)
 			(effects
@@
 	)
 	(sheet
-		(at 302.26 151.13)
-		(size 34.29 17.78)
+		(at 293.37 152.4)
+		(size 43.18 17.78)
 		(exclude_from_sim no)
 		(in_bom yes)
@@
 			(color 0 0 0 0.0000)
 		)
-		(property "Sheetname" "Nixie Driver"
-			(at 302.26 150.4184 0)
+		(property "Sheetname" "HV PSU"
+			(at 293.37 151.6884 0)
 			(effects
 				(font
@@
 			)
 		)
-		(property "Sheetfile" "sch/nixie_driver.kicad_sch"
-			(at 302.26 169.4946 0)
+		(property "Sheetfile" "sch/hv_psu.kicad_sch"
+			(at 293.37 170.7646 0)
 			(effects
 				(font
@@
 			)
 		)
-		(pin "G_A[0..5]" bidirectional
-			(at 302.26 160.02 180)
-			(effects
-				(font
-					(size 1.27 1.27)
-				)
-				(justify left)
-			)
-		)
-		(pin "N[0..3]" bidirectional
-			(at 302.26 157.48 180)
-			(effects
-				(font
-					(size 1.27 1.27)
-				)
-				(justify left)
-			)
-		)
-		(pin "~{N_LE}" bidirectional
-			(at 302.26 162.56 180)
-			(effects
-				(font
-					(size 1.27 1.27)
-				)
-				(justify left)
-			)
-		)
 		(instances
-			(project "Yet-Another-Nixie-Clock"
+			(project "Yet-Another-Nixie-Clock-Processing"
 				(path "/78ce616d-4594-460a-a6b5-d8dd90d9a741"
-					(page "4")
+					(page "2")
 				)
 			)

Commit message: Major schematic and layout advancements
Parts:
- removed D1: Green, LED_SMD:LED_0603_1608Metric, symbol Device:LED
- removed D15: LED, LED_SMD:LED_0603_1608Metric, symbol Device:LED
- removed H1, H4: MountingHole_Pad, MountingHole:MountingHole_3.2mm_M3_Pad, symbol Mechanical:MountingHole_Pad
- removed R16: 0, Resistor_SMD:R_0402_1005Metric, symbol Device:R_Small_US
- removed R8: 1k, symbol Device:R_Small_US
- added D4: LED, LED_SMD:LED_0603_1608Metric, symbol Device:LED
- added R21: 1k, Resistor_SMD:R_0603_1608Metric, symbol Device:R_Small_US
- BT1: footprint (none) -> Yet-Another-Nixie-Clock-Face:BAT-TH_CR2032-BS-6-1
- J3: footprint (none) -> Connector_IDC:IDC-Header_2x05_P2.54mm_Vertical
- R1, R10, R11, R12, R13, R17, R2, R3, R6, R7, R9: footprint (none) -> Resistor_SMD:R_0603_1608Metric
- R14, R15: footprint Resistor_SMD:R_0402_1005Metric -> Resistor_SMD:R_0603_1608Metric
- SW1, SW2, SW3: footprint Yet-Another-Nixie-Clock-Processing:SW_SKRPACE010 -> Yet-Another-Nixie-Clock:SW_SKRPACE010
Connections:
- net CP_3V3: now also R9.1, R21.1
- net GND: no longer D2.1 (K), J10.12 (Pin_12)
- net G_A0: now also J10.2 (Pin_2), U5.26 (IO4); no longer J10.1 (Pin_1), U5.10 (IO25)
- net G_A1: now also J10.4 (Pin_4), U5.27 (IO16); no longer J10.3 (Pin_3), U5.11 (IO26)
- net G_A2: now also J10.6 (Pin_6); no longer J10.5 (Pin_5)
- net G_A3: now also J10.8 (Pin_8), U5.10 (IO25); no longer J10.7 (Pin_7), U5.8 (IO32)
- net G_A4: now also J10.10 (Pin_10), U5.8 (IO32); no longer J10.9 (Pin_9), U5.9 (IO33)
- net G_A5: now also J10.1 (Pin_1), U5.28 (IO17); no longer J10.2 (Pin_2), U5.6 (IO34)
- net LED_1: now also J10.11 (Pin_11), U5.6 (IO34); no longer R9.1, U5.26 (IO4)
- net N0: now also J10.3 (Pin_3), U5.30 (IO18); no longer J10.4 (Pin_4), U5.27 (IO16)
- net N1: now also J10.5 (Pin_5), U5.31 (IO19); no longer J10.6 (Pin_6), U5.28 (IO17)
- net N2: now also J10.7 (Pin_7), U5.11 (IO26); no longer J10.8 (Pin_8), U5.30 (IO18)
- net N3: now also J10.9 (Pin_9), U5.9 (IO33); no longer J10.10 (Pin_10), U5.31 (IO19)
- net VCC3V3: now also J11.7 (Pin_7), J11.8 (Pin_8)
- net ~{N_LE}: now also J10.12 (Pin_12); no longer J10.11 (Pin_11)
- net at U1.13 (~{RXT}/GPIO.1): now also D4.1 (K)
- net at U1.14 (~{TXT}/GPIO.0): now also D2.1 (K)
- new net: D4.2 (A), R21.2
- no-connect marks 7 -> 6
Other:
- moved on the sheet: C4, C6, C7, C8

Commit message: Minor touches. Fixed bom. Exported production files
Parts:
- BT1, D16, D17, D2, D4: now left out of the parts list
- J10, J11: LCSC (none) -> C2685123
- J3: LCSC (none) -> C573025
- Q1, Q2: LCSC (none) -> C82460
- R14, R15: LCSC (none) -> C99782
- U2: LCSC (none) -> C97253
- U4: LCSC (none) -> C722467
- U5: LCSC (none) -> C82899
Changed lines of the file:
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@@
 		(unit 1)
 		(exclude_from_sim no)
-		(in_bom yes)
+		(in_bom no)
 		(on_board yes)
 		(dnp no)
@@
 		(unit 1)
 		(exclude_from_sim no)
-		(in_bom yes)
+		(in_bom no)
 		(on_board yes)
 		(dnp no)
@@
 			)
 		)
+		(property "LCSC" "C2685123"
+			(at 370.84 162.56 0)
+			(effects
+				(font
+					(size 1.27 1.27)
+				)
+				(hide yes)
+			)
+		)
 		(pin "12"
 		)
@@
 			)
 		)
+		(property "LCSC" "C2685123"
+			(at 257.81 160.02 0)
+			(effects
+				(font
+					(size 1.27 1.27)
+				)
+				(hide yes)
+			)
+		)
 		(pin "6"
 		)
@@
 			)
 		)
-		(property "LCSC" ""
+		(property "LCSC" "C99782"
 			(at 279.4 207.01 0)
 			(effects
@@
 			)
 		)
+		(property "LCSC" "C82460"
+			(at 55.88 138.43 0)
+			(effects
+				(font
+					(size 1.27 1.27)
+				)
+				(hide yes)
+			)
+		)
 		(pin "2"
 		)
@@
 		(unit 1)
 		(exclude_from_sim no)
-		(in_bom yes)
+		(in_bom no)
 		(on_board yes)
 		(dnp no)
@@
 		(unit 1)
 		(exclude_from_sim no)
-		(in_bom yes)
+		(in_bom no)
 		(on_board yes)
 		(dnp no)
@@
 		(unit 1)
 		(exclude_from_sim no)
-		(in_bom yes)
+		(in_bom no)
 		(on_board yes)
 		(dnp no)
@@
 			)
 		)
+		(property "LCSC" "C82460"
+			(at 55.88 121.92 0)
+			(effects
+				(font
+					(size 1.27 1.27)
+				)
+				(hide yes)
+			)
+		)
 		(pin "2"
 		)
@@
 			)
 		)
+		(property "LCSC" "C573025"
+			(at 374.65 43.18 0)
+			(effects
+				(font
+					(size 1.27 1.27)
+				)
+				(hide yes)
+			)
+		)
 		(pin "4"
 		)
@@
 			)
 		)
+		(property "LCSC" "C82899"
+			(at 308.61 69.85 0)
+			(effects
+				(font
+					(size 1.27 1.27)
+				)
+				(hide yes)
+			)
+		)
 		(pin "23"
 		)
@@
 			)
 		)
+		(property "LCSC" "C722467"
+			(at 300.99 220.98 0)
+			(effects
+				(font
+					(size 1.27 1.27)
+				)
+				(hide yes)
+			)
+		)
 		(pin "14"
 		)
@@
 			)
 		)
+		(property "LCSC" "C97253"
+			(at 104.14 36.83 0)
+			(effects
+				(font
+					(size 1.27 1.27)
+				)
+				(hide yes)
+			)
+		)
 		(pin "4"
 		)
@@
 			)
 		)
-		(property "LCSC" ""
+		(property "LCSC" "C99782"
 			(at 284.48 207.01 0)
 			(effects
