File: Hardware/Yet-Another-Nixie-Clock-Processing/sch/hv_psu.kicad_sch (KiCad schematic)
At the start: 13 parts, among them Q3 Q_NMOS, U6 MAX1771xSA

Commit message: Minor touches. Fixed bom. Exported production files
Parts:
- U6: LCSC (none) -> C407903
Changed lines of the file:
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@@
+			)
+		)
+		(property "LCSC" "C407903"
+			(at 120.65 93.98 0)
+			(effects
+				(font
+					(size 1.27 1.27)
+				)
+				(hide yes)
 			)
 		)
